Commit message: updated inertias

File: mico_description/urdf/arms/mico_arm.gazebo.xacro (robot description, xacro)
@@ -16,33 +16,33 @@
 	</gazebo>
 	<gazebo reference="mico_link_1">
-		<material>Gazebo/Black</material>
+		<material>Gazebo/FlatBlack</material>
 		<turnGravityOff>true</turnGravityOff>
 	</gazebo>
 	<gazebo reference="mico_link_2">
-		<material>Gazebo/Black</material>
+		<material>Gazebo/FlatBlack</material>
 		<turnGravityOff>true</turnGravityOff>
 	</gazebo>
 	<gazebo reference="mico_link_3">
-		<material>Gazebo/Black</material>
+		<material>Gazebo/FlatBlack</material>
 		<turnGravityOff>true</turnGravityOff>
 	</gazebo>
 	<gazebo reference="mico_link_4">
-		<material>Gazebo/Black</material>
+		<material>Gazebo/FlatBlack</material>
 		<turnGravityOff>true</turnGravityOff>
 	</gazebo>
 	<gazebo reference="mico_link_5">
-		<material>Gazebo/Black</material>
+		<material>Gazebo/FlatBlack</material>
 		<turnGravityOff>true</turnGravityOff>
 	</gazebo>
 	<gazebo reference="mico_link_hand">
-		<material>Gazebo/Black</material>
+		<material>Gazebo/FlatBlack</material>
 		<turnGravityOff>true</turnGravityOff>
 	</gazebo>
 	<gazebo reference="mico_link_finger_1">
-		<material>Gazebo/Gray</material>
+		<material>Gazebo/Grey</material>
 		<turnGravityOff>true</turnGravityOff>
 	</gazebo>
 	<gazebo reference="mico_link_finger_2">
-		<material>Gazebo/Gray</material>
+		<material>Gazebo/Grey</material>
 		<turnGravityOff>true</turnGravityOff>
 	</gazebo>

File: mico_description/urdf/arms/mico_arm.urdf.xacro (robot description, xacro)
@@ -178,7 +178,7 @@
 	<link name="mico_link_3">
 		<inertial>
-		  <mass value="0.429" />
-		  <origin xyz="0.06076 0 -0.00014" />
-		  <inertia  ixx="0.0011551458" ixy="-6.3e-010"  ixz="2.519546e-005"  iyy="0.0015754353"  iyz="-7.6e-010"  izz="0.0007798411" />
+		  <mass value="0.351" />
+		  <origin xyz="-0.07306 0 -0.00466" />
+		  <inertia  ixx="0.0003749308" ixy="0.0"  ixz="-0.0001258961"  iyy="0.0010047174"  iyz="0.0"  izz="0.0009318091" />
 		</inertial>
 		<visual>
@@ -383,5 +383,5 @@
 		<inertial>
 		  <mass value="0.050" />
-		  <origin xyz="0.01 0.01 0.01" />
+		  <origin xyz="0.03 0.03 0.03" />
 		  <inertia  ixx="0.0011551458" ixy="-6.3e-010"  ixz="2.519546e-005"  iyy="0.0015754353"  iyz="-7.6e-010"  izz="0.0007798411" />
 		</inertial>
@@ -434,5 +434,5 @@
 		<inertial>
 		  <mass value="0.050" />
-		  <origin xyz="0.01 0.01 0.01" />
+		  <origin xyz="0.03 0.03 0.03" />
 		  <inertia  ixx="0.0011551458" ixy="-6.3e-010"  ixz="2.519546e-005"  iyy="0.0015754353"  iyz="-7.6e-010"  izz="0.0007798411" />
 		</inertial>
