Commit message: changed joint names to those used by the jaco_ros driver

File: mico_description/urdf/arms/mico_arm.urdf.xacro (robot description, xacro)
@@ -104,5 +104,5 @@
 	</link>
 	<joint
-		name="j1"
+		name="mico_joint_1"
 		type="revolute">
 		<origin
@@ -117,5 +117,5 @@
     <transmission name="j1_trans">
 	 <type>transmission_interface/SimpleTransmission</type>
-     <joint name="j1" />
+     <joint name="mico_joint_1" />
      <actuator name="j1_motor">
 	    <hardwareInterface>EffortJointInterface</hardwareInterface>
@@ -155,5 +155,5 @@
 	</link>
 	<joint
-		name="j2"
+		name="mico_joint_2"
 		type="revolute">
 	  <origin
@@ -168,5 +168,5 @@
     <transmission name="j2_trans">
 	 <type>transmission_interface/SimpleTransmission</type>
-     <joint name="j2" />
+     <joint name="mico_joint_2" />
      <actuator name="j2_motor">
 	    <hardwareInterface>EffortJointInterface</hardwareInterface>
@@ -206,5 +206,5 @@
 	</link>
 	<joint
-		name="j3"
+		name="mico_joint_3"
 		type="revolute">
 	  <origin
@@ -219,5 +219,5 @@
     <transmission name="j3_trans">
 	 <type>transmission_interface/SimpleTransmission</type>
-     <joint name="j3" />
+     <joint name="mico_joint_3" />
      <actuator name="j3_motor">
 	    <hardwareInterface>EffortJointInterface</hardwareInterface>
@@ -257,5 +257,5 @@
 	</link>
 	<joint
-		name="j4"
+		name="mico_joint_4"
 		type="revolute">
 	  <origin
@@ -270,5 +270,5 @@
     <transmission name="j4_trans">
 	 <type>transmission_interface/SimpleTransmission</type>
-     <joint name="j4" />
+     <joint name="mico_joint_4" />
      <actuator name="j4_motor">
 	    <hardwareInterface>EffortJointInterface</hardwareInterface>
@@ -308,5 +308,5 @@
 	</link>
 	<joint
-		name="j5"
+		name="mico_joint_5"
 		type="revolute">
 	  <origin
@@ -321,5 +321,5 @@
     <transmission name="j5_trans">
 	 <type>transmission_interface/SimpleTransmission</type>
-     <joint name="j5" />
+     <joint name="mico_joint_5" />
      <actuator name="j5_motor">
 	    <hardwareInterface>EffortJointInterface</hardwareInterface>
@@ -359,5 +359,5 @@
 	</link>
 	<joint
-		name="j6"
+		name="mico_joint_6"
 		type="revolute">
 	  <origin
@@ -372,5 +372,5 @@
     <transmission name="j6_trans">
 	 <type>transmission_interface/SimpleTransmission</type>
-     <joint name="j6" />
+     <joint name="mico_joint_6" />
      <actuator name="j6_motor">
 	    <hardwareInterface>EffortJointInterface</hardwareInterface>
@@ -410,5 +410,5 @@
 	</link>
 	<joint
-		name="jf1"
+		name="mico_joint_finger_1"
 		type="revolute">
 	  <origin
@@ -423,5 +423,5 @@
     <transmission name="jf1_trans">
 	 <type>transmission_interface/SimpleTransmission</type>
-     <joint name="jf1" />
+     <joint name="mico_joint_finger_1" />
      <actuator name="jf1_motor">
 	    <hardwareInterface>EffortJointInterface</hardwareInterface>
@@ -461,5 +461,5 @@
 	</link>
 	<joint
-		name="jf2"
+		name="mico_joint_finger_2"
 		type="revolute">
 	  <origin
@@ -474,5 +474,5 @@
     <transmission name="jf2_trans">
 	 <type>transmission_interface/SimpleTransmission</type>
-     <joint name="jf2" />
+     <joint name="mico_joint_finger_2" />
      <actuator name="jf2_motor">
 	    <hardwareInterface>EffortJointInterface</hardwareInterface>
